Commit message: added Hokuyo rangefinder mesh

File: mybot_description/urdf/mybot.xacro (robot description, xacro)
@@ -185,5 +185,5 @@
       <origin xyz="0 0 0" rpy="0 0 0"/>
       <geometry>
-        <box size="0.001 0.001 0.001"/>
+        <mesh filename="$(find mybot_description)/meshes/hokuyo.dae" />
       </geometry>
     </visual>

Commit message: modified mesh filepath to be visible for RViz

File: mybot_description/urdf/mybot.xacro (robot description, xacro)
@@ -4,5 +4,5 @@
   <xacro:property name="cameraMass" value="0.1"/>
   <xacro:include filename="$(find mybot_description)/urdf/mybot.gazebo" />
-  <xacro:include filename="$(find mybot_description)/urdf/materials.xacro" />
+  <!-- <xacro:include filename="$(find mybot_description)/urdf/materials.xacro" /> -->
   <xacro:include filename="$(find mybot_description)/urdf/macros.xacro" />
   <link name='chassis'>
@@ -25,8 +25,7 @@
       <origin xyz="0.5348 0.21 -0.252" rpy=" 0 0 -1.57"/>
       <geometry>
-        <mesh
-          filename="$(find mybot_description)/meshes/chassis.STL" />
+        <mesh filename="package://mybot_description/meshes/chassis.STL" />
       </geometry>
-<material name="black"/>
+<!-- <material name="orange"/> -->
     </visual>
     <collision name='caster_collision'>
@@ -86,6 +85,5 @@
       <origin xyz="0 0.027 0" rpy="1.57 0 0"/>
        <geometry>
-        <mesh
-          filename="$(find mybot_description)/meshes/lwheel.STL" />
+        <mesh filename="package://mybot_description/meshes/lwheel.STL" />
       </geometry>
     </visual>
@@ -110,6 +108,5 @@
       <origin xyz="0 -0.1 0" rpy="1.57 0 0"/>
        <geometry>
-        <mesh
-          filename="$(find mybot_description)/meshes/rwheel.STL" />
+        <mesh filename="package://mybot_description/meshes/rwheel.STL" />
       </geometry>
     </visual>
@@ -153,5 +150,5 @@
          <box size="0.001 0.001 0.001"/>
       </geometry>
-      <material name="green"/>
+      <!-- <material name="green"/> -->
     </visual>
     <inertial>
@@ -185,5 +182,5 @@
       <origin xyz="0 0 0" rpy="0 0 0"/>
       <geometry>
-        <mesh filename="$(find mybot_description)/meshes/hokuyo.dae" />
+        <mesh filename="package://mybot_description/meshes/hokuyo.dae" />
       </geometry>
     </visual>

Commit message: feat: Add RPLIDAR

File: mybot_description/urdf/mybot.xacro (robot description, xacro)
@@ -6,4 +6,12 @@
   <!-- <xacro:include filename="$(find mybot_description)/urdf/materials.xacro" /> -->
   <xacro:include filename="$(find mybot_description)/urdf/macros.xacro" />
+  <link name="base_link">
+  </link>
+  <joint name="base_joint" type="fixed">
+    <axis xyz="0 0 0" />
+    <origin xyz="0 0 0" rpy="0 0 0"/>
+    <parent link="base_link"/>
+    <child link="chassis"/>
+  </joint>
   <link name='chassis'>
     <pose>0 0 0.1 0 0 0</pose>
@@ -165,29 +173,29 @@
     <child link="camera"/>
   </joint>
-  <joint name="hokuyo_joint" type="fixed">
+  <!-- rplidar Laser -->
+  <link name="rplidar">
+    <collision>
+      <origin xyz="0 0 0" rpy="0 0 0"/>
+      <geometry>
+    <box size="0.1 0.1 0.1"/>
+      </geometry>
+    </collision>
+    <visual>
+      <origin xyz="0 0 0" rpy="0 0 0"/>
+      <geometry>
+        <mesh filename="package://mybot_description/meshes/rplidar.dae" />
+      </geometry>
+    </visual>
+    <inertial>
+      <mass value="1e-5" />
+      <origin xyz="0 0 0" rpy="0 0 0"/>
+      <inertia ixx="1e-6" ixy="0" ixz="0" iyy="1e-6" iyz="0" izz="1e-6" />
+    </inertial>
+  </link>
+  <joint name="rplidar_joint" type="fixed">
     <axis xyz="0 1 0" />
     <origin xyz=".15 0 .2" rpy="0 0 0"/>
     <parent link="chassis"/>
-    <child link="hokuyo"/>
-  </joint>
-  <!-- Hokuyo Laser -->
-  <link name="hokuyo">
-    <collision>
-      <origin xyz="0 0 0" rpy="0 0 0"/>
-      <geometry>
-    <box size="0.1 0.1 0.1"/>
-      </geometry>
-    </collision>
-    <visual>
-      <origin xyz="0 0 0" rpy="0 0 0"/>
-      <geometry>
-        <mesh filename="package://mybot_description/meshes/hokuyo.dae" />
-      </geometry>
-    </visual>
-    <inertial>
-      <mass value="1e-5" />
-      <origin xyz="0 0 0" rpy="0 0 0"/>
-      <inertia ixx="1e-6" ixy="0" ixz="0" iyy="1e-6" iyz="0" izz="1e-6" />
-    </inertial>
-  </link>
+    <child link="rplidar"/>
+  </joint>
 </robot>
